Commit message: save

File: catkin_ws/src/kit_agv_description/urdf/kit_agv.urdf.xacro (robot description, xacro)
@@ -17,5 +17,5 @@
     <parent link="base_link"/>
     <child link="base_laser"/>
-    <origin xyz="0.369 -0.21335 0.059" rpy="0 0 0"/>
+    <origin xyz="0.266717 0 0.156017" rpy="0 0 0"/>
   </joint>
   <link name="wheel_right_link">
